Commit message: add commander and service msgs

File: turtlebot3_description/urdf/turtlebot3_covid.gazebo.xacro (robot description, xacro)
@@ -2,5 +2,5 @@
 <robot name="robot_covid_sim" xmlns:xacro="http://ros.org/wiki/xacro">
   <xacro:arg name="laser_visual"  default="false"/>
-  <xacro:arg name="camera_visual" default="false"/>
+  <!-- <xacro:arg name="camera_visual" default="false"/> -->
   <xacro:arg name="imu_visual"    default="false"/>
   <gazebo reference="base_link">
@@ -153,5 +153,5 @@
   </gazebo>
 <!--link : https://www.raspberrypi.org/documentation/hardware/camera/-->
-  <gazebo reference="camera_rgb_frame">
+  <!-- <gazebo reference="camera_rgb_frame">
     <sensor type="camera" name="Pi Camera">
       <always_on>true</always_on>
@@ -184,4 +184,4 @@
       </plugin>
     </sensor>
-  </gazebo>
+  </gazebo> -->
 </robot>

File: turtlebot3_description/urdf/turtlebot3_covid.urdf.xacro (robot description, xacro)
@@ -3,4 +3,5 @@
   <xacro:include filename="$(find turtlebot3_description)/urdf/common_properties.xacro"/>
   <xacro:include filename="$(find turtlebot3_description)/urdf/turtlebot3_covid.gazebo.xacro"/>
+  <xacro:include filename="$(find realsense2_description)/urdf/_d435.urdf.xacro" />
   <link name="base_footprint"/>
   <joint name="base_joint" type="fixed">
@@ -788,5 +789,5 @@
     <parent link="base_link"/>
     <child link="base_scan"/>
-    <origin xyz="-0.40 0 0.93" rpy="0 0 3.14"/>
+    <origin xyz="-0.35 0 0.93" rpy="0 0 3.14"/>
   </joint>
   <link name="base_scan">
@@ -812,5 +813,8 @@
     </inertial>
   </link>
-  <joint name="camera_joint" type="fixed">
+  <sensor_d435 parent="base_link">
+    <origin xyz="-0.32 0 0.83" rpy="0 0 0"/>
+  </sensor_d435>
+  <!-- <joint name="camera_joint" type="fixed">
     <origin xyz="-0.35 0 0.83" rpy="0 0 0"/>
     <parent link="base_link"/>
@@ -836,4 +840,4 @@
     <child link="camera_rgb_optical_frame"/>
   </joint>
-  <link name="camera_rgb_optical_frame"/>
+  <link name="camera_rgb_optical_frame"/> -->
 </robot>
