Commit message: update urdf stl reference

File: turtlebot3_description/urdf/turtlebot3_covid.urdf.xacro (robot description, xacro)
@@ -31,5 +31,5 @@
       <geometry>
         <mesh
-          filename="package://robot_covid/meshes/base_link.STL" />
+          filename="package://turtlebot3_description/meshes/base_link.STL" />
       </geometry>
       <material
@@ -45,5 +45,5 @@
       <geometry>
         <mesh
-          filename="package://robot_covid/meshes/base_link.STL" />
+          filename="package://turtlebot3_description/meshes/base_link.STL" />
       </geometry>
     </collision>
@@ -71,5 +71,5 @@
       <geometry>
         <mesh
-          filename="package://robot_covid/meshes/right_wheel.STL" />
+          filename="package://turtlebot3_description/meshes/right_wheel.STL" />
       </geometry>
       <material
@@ -85,5 +85,5 @@
       <geometry>
         <mesh
-          filename="package://robot_covid/meshes/right_wheel.STL" />
+          filename="package://turtlebot3_description/meshes/right_wheel.STL" />
       </geometry>
     </collision>
@@ -137,5 +137,5 @@
       <geometry>
         <mesh
-          filename="package://robot_covid/meshes/left_wheel.STL" />
+          filename="package://turtlebot3_description/meshes/left_wheel.STL" />
       </geometry>
       <material
@@ -151,5 +151,5 @@
       <geometry>
         <mesh
-          filename="package://robot_covid/meshes/left_wheel.STL" />
+          filename="package://turtlebot3_description/meshes/left_wheel.STL" />
       </geometry>
     </collision>
@@ -203,5 +203,5 @@
       <geometry>
         <mesh
-          filename="package://robot_covid/meshes/caster_right_front.STL" />
+          filename="package://turtlebot3_description/meshes/caster_right_front.STL" />
       </geometry>
       <material
@@ -217,5 +217,5 @@
       <geometry>
         <mesh
-          filename="package://robot_covid/meshes/caster_right_front.STL" />
+          filename="package://turtlebot3_description/meshes/caster_right_front.STL" />
       </geometry>
     </collision>
@@ -261,5 +261,5 @@
       <geometry>
         <mesh
-          filename="package://robot_covid/meshes/caster_wheel_right_front.STL" />
+          filename="package://turtlebot3_description/meshes/caster_wheel_right_front.STL" />
       </geometry>
       <material
@@ -275,5 +275,5 @@
       <geometry>
         <mesh
-          filename="package://robot_covid/meshes/caster_wheel_right_front.STL" />
+          filename="package://turtlebot3_description/meshes/caster_wheel_right_front.STL" />
       </geometry>
     </collision>
@@ -322,5 +322,5 @@
       <geometry>
         <mesh
-          filename="package://robot_covid/meshes/caster_left_front.STL" />
+          filename="package://turtlebot3_description/meshes/caster_left_front.STL" />
       </geometry>
       <material
@@ -336,5 +336,5 @@
       <geometry>
         <mesh
-          filename="package://robot_covid/meshes/caster_left_front.STL" />
+          filename="package://turtlebot3_description/meshes/caster_left_front.STL" />
       </geometry>
     </collision>
@@ -380,5 +380,5 @@
       <geometry>
         <mesh
-          filename="package://robot_covid/meshes/caster_wheel_left_front.STL" />
+          filename="package://turtlebot3_description/meshes/caster_wheel_left_front.STL" />
       </geometry>
       <material
@@ -394,5 +394,5 @@
       <geometry>
         <mesh
-          filename="package://robot_covid/meshes/caster_wheel_left_front.STL" />
+          filename="package://turtlebot3_description/meshes/caster_wheel_left_front.STL" />
       </geometry>
     </collision>
@@ -441,5 +441,5 @@
       <geometry>
         <mesh
-          filename="package://robot_covid/meshes/caster_right_rear.STL" />
+          filename="package://turtlebot3_description/meshes/caster_right_rear.STL" />
       </geometry>
       <material
@@ -455,5 +455,5 @@
       <geometry>
         <mesh
-          filename="package://robot_covid/meshes/caster_right_rear.STL" />
+          filename="package://turtlebot3_description/meshes/caster_right_rear.STL" />
       </geometry>
     </collision>
@@ -499,5 +499,5 @@
       <geometry>
         <mesh
-          filename="package://robot_covid/meshes/caster_wheel_right_rear.STL" />
+          filename="package://turtlebot3_description/meshes/caster_wheel_right_rear.STL" />
       </geometry>
       <material
@@ -513,5 +513,5 @@
       <geometry>
         <mesh
-          filename="package://robot_covid/meshes/caster_wheel_right_rear.STL" />
+          filename="package://turtlebot3_description/meshes/caster_wheel_right_rear.STL" />
       </geometry>
     </collision>
@@ -560,5 +560,5 @@
       <geometry>
         <mesh
-          filename="package://robot_covid/meshes/caster_left_rear.STL" />
+          filename="package://turtlebot3_description/meshes/caster_left_rear.STL" />
       </geometry>
       <material
@@ -574,5 +574,5 @@
       <geometry>
         <mesh
-          filename="package://robot_covid/meshes/caster_left_rear.STL" />
+          filename="package://turtlebot3_description/meshes/caster_left_rear.STL" />
       </geometry>
     </collision>
@@ -618,5 +618,5 @@
       <geometry>
         <mesh
-          filename="package://robot_covid/meshes/caster_wheel_left_rear.STL" />
+          filename="package://turtlebot3_description/meshes/caster_wheel_left_rear.STL" />
       </geometry>
       <material
@@ -632,5 +632,5 @@
       <geometry>
         <mesh
-          filename="package://robot_covid/meshes/caster_wheel_left_rear.STL" />
+          filename="package://turtlebot3_description/meshes/caster_wheel_left_rear.STL" />
       </geometry>
     </collision>
@@ -657,4 +657,126 @@
       k_velocity="1" />
   </joint>
+  <link
+    name="panel_tower">
+    <inertial>
+      <origin
+        xyz="0.0064322 -0.0025126 0.03"
+        rpy="0 0 0" />
+      <mass
+        value="12.15" />
+      <inertia
+        ixx="0.57318"
+        ixy="4.2001E-17"
+        ixz="5.0155E-20"
+        iyy="0.00729"
+        iyz="7.3794E-18"
+        izz="0.57318" />
+    </inertial>
+    <visual>
+      <origin
+        xyz="0 0 0"
+        rpy="0 0 0" />
+      <geometry>
+        <mesh
+          filename="package://turtlebot3_description/meshes/panel_tower.STL" />
+      </geometry>
+      <material
+        name="">
+        <color
+          rgba="0.68627 0.65882 0.63922 1" />
+      </material>
+    </visual>
+    <collision>
+      <origin
+        xyz="0 0 0"
+        rpy="0 0 0" />
+      <geometry>
+        <mesh
+          filename="package://turtlebot3_description/meshes/panel_tower.STL" />
+      </geometry>
+    </collision>
+  </link>
+  <joint
+    name="base_panel_tower"
+    type="fixed">
+    <origin
+      xyz="-0.42643 0.03 0.37751"
+      rpy="1.5708 0 0" />
+    <parent
+      link="base_link" />
+    <child
+      link="panel_tower" />
+    <axis
+      xyz="0 0 0" />
+    <limit
+      effort="10000"
+      velocity="0" />
+    <dynamics
+      damping="1000"
+      friction="1000" />
+    <safety_controller
+      k_velocity="1" />
+  </joint>
+  <link
+    name="panel_housing">
+    <inertial>
+      <origin
+        xyz="-0.0089661 0.1507 0.017336"
+        rpy="0 0 0" />
+      <mass
+        value="9.8248" />
+      <inertia
+        ixx="0.10476"
+        ixy="0.00014166"
+        ixz="0.0062239"
+        iyy="0.034911"
+        iyz="0.00014628"
+        izz="0.094801" />
+    </inertial>
+    <visual>
+      <origin
+        xyz="0 0 0"
+        rpy="0 0 0" />
+      <geometry>
+        <mesh
+          filename="package://turtlebot3_description/meshes/panel_housing.STL" />
+      </geometry>
+      <material
+        name="">
+        <color
+          rgba="0.68627 0.65882 0.63922 1" />
+      </material>
+    </visual>
+    <collision>
+      <origin
+        xyz="0 0 0"
+        rpy="0 0 0" />
+      <geometry>
+        <mesh
+          filename="package://turtlebot3_description/meshes/panel_housing.STL" />
+      </geometry>
+    </collision>
+  </link>
+  <joint
+    name="base_panel_housing"
+    type="fixed">
+    <origin
+      xyz="-0.37982 0.14882 0.82388"
+      rpy="3.1416 0 0" />
+    <parent
+      link="base_link" />
+    <child
+      link="panel_housing" />
+    <axis
+      xyz="0 0 0" />
+    <limit
+      effort="10000"
+      velocity="0" />
+    <dynamics
+      damping="1000"
+      friction="1000" />
+    <safety_controller
+      k_velocity="1" />
+  </joint>
   <joint name="imu_joint" type="fixed">
     <parent link="base_link"/>
@@ -666,5 +788,5 @@
     <parent link="base_link"/>
     <child link="base_scan"/>
-    <origin xyz="-0.47 0 0.93" rpy="0 0 0"/>
+    <origin xyz="-0.40 0 0.93" rpy="0 0 0"/>
   </joint>
   <link name="base_scan">

Commit message: change lidar scan orientaion

File: turtlebot3_description/urdf/turtlebot3_covid.urdf.xacro (robot description, xacro)
@@ -782,5 +782,5 @@
     <parent link="base_link"/>
     <child link="imu_link"/>
-    <origin xyz="0.0 0 0.068" rpy="0 0 0"/>
+    <origin xyz="-0.34 0 0.068" rpy="0 0 0"/>
   </joint>
   <link name="imu_link"/>
@@ -788,5 +788,5 @@
     <parent link="base_link"/>
     <child link="base_scan"/>
-    <origin xyz="-0.40 0 0.93" rpy="0 0 0"/>
+    <origin xyz="-0.40 0 0.93" rpy="0 0 3.14"/>
   </joint>
   <link name="base_scan">
@@ -813,5 +813,5 @@
   </link>
   <joint name="camera_joint" type="fixed">
-    <origin xyz="0.073 -0.011 0.084" rpy="0 0 0"/>
+    <origin xyz="-0.35 0 0.83" rpy="0 0 0"/>
     <parent link="base_link"/>
     <child link="camera_link"/>

Commit message: move state publisher to covid robot

File: turtlebot3_description/urdf/turtlebot3_covid.urdf.xacro (robot description, xacro)
@@ -8,5 +8,5 @@
     <parent link="base_footprint"/>
     <child link="base_link" />
-    <origin xyz="0 0 0" rpy="0 0 0"/>
+    <origin xyz="0 0 0" rpy="0 0 3.14"/>
   </joint>
   <link
@@ -51,5 +51,5 @@
   </link>
   <link
-    name="right_wheel">
+    name="left_wheel">
     <inertial>
       <origin
@@ -91,5 +91,5 @@
   </link>
   <joint
-    name="wheel_right_joint"
+    name="wheel_left_joint"
     type="continuous">
     <origin
@@ -99,5 +99,5 @@
       link="base_link" />
     <child
-      link="right_wheel" />
+      link="left_wheel" />
     <axis
       xyz="0 0 1" />
@@ -117,5 +117,5 @@
   </joint>
   <link
-    name="left_wheel">
+    name="right_wheel">
     <inertial>
       <origin
@@ -157,5 +157,5 @@
   </link>
   <joint
-    name="wheel_left_joint"
+    name="wheel_right_joint"
     type="continuous">
     <origin
@@ -165,5 +165,5 @@
       link="base_link" />
     <child
-      link="left_wheel" />
+      link="right_wheel" />
     <axis
       xyz="0 0 -1" />
@@ -789,5 +789,5 @@
     <parent link="base_link"/>
     <child link="base_scan"/>
-    <origin xyz="-0.35 0 0.93" rpy="0 0 3.14"/>
+    <origin xyz="-0.35 0 0.93" rpy="0 0 0"/>
   </joint>
   <link name="base_scan">
@@ -814,5 +814,5 @@
   </link>
   <sensor_d435 parent="base_link">
-    <origin xyz="-0.32 0 0.83" rpy="0 0 0"/>
+    <origin xyz="-0.38 0 0.83" rpy="0 0 3.14"/>
   </sensor_d435>
   <!-- <joint name="camera_joint" type="fixed">
